File: cr432/assemble/assemble.kicad_pcb (KiCad board)
At the start: 2 copper layers, 229.6 x 78.6 mm, 102 parts, among them SW1 SW_Push, SW10 SW_Push, SW11 SW_Push, SW12 SW_Push, SW13 SW_Push, SW14 SW_Push, SW15 SW_Push, SW16 SW_Push, SW17 SW_Push, SW18 SW_Push, SW19 SW_Push, SW2 SW_Push, SW20 SW_Push, SW21 SW_Push, SW22 SW_Push, SW23 SW_Push, SW24 SW_Push, SW25 SW_Push, SW26 SW_Push, SW27 SW_Push, SW28 SW_Push, SW29 SW_Push, SW3 SW_Push, SW30 SW_Push, SW31 SW_Push, SW32 SW_Push, SW33 SW_Push, SW34 SW_Push, SW35 SW_Push, SW36 SW_Push, SW37 SW_Push, SW38 SW_Push, SW39 SW_Push, SW4 SW_Push, SW40 SW_Push, SW41 SW_Push, SW42 SW_Push, SW43 SW_Push, SW44 SW_Push, SW5 SW_Push, SW6 SW_Push, SW7 SW_Push, SW8 SW_Push, SW9 SW_Push, U1 Micon_BLEMicroPro

Commit message: rev1
Parts:
- removed the D40 at (263.0, 92.0)
- removed the D42 at (266.7, 53.8)
- removed the Ref** at (126.2, 79.3)
- removed the Ref** at (80.2, 42.1)
- removed the Ref** at (193.8, 42.1)
- removed the Ref** at (257.2, 115.0)
- removed the Ref** at (183.4, 79.3)
- removed the Ref** at (202.4, 115.0)
- removed the Ref** at (117.6, 42.1)
- removed the Ref** at (83.3, 77.9)
- removed the Ref** at (266.7, 95.2)
- removed the Ref** at (52.4, 115.0)
- removed the Ref** at (235.7, 77.9)
- removed the Ref** at (251.7, 42.1)
- removed the Ref** at (107.2, 115.0)
- removed the Ref** at (42.9, 95.2)
- removed the SW41 at (254.8, 88.1)
- added D41: D, kbd_Parts:Diode_SMD, F.Cu at (253.8, 70.1)
- added D43: D, kbd_Parts:Diode_SMD, F.Cu at (272.9, 51.0)
- added D44: D, kbd_Parts:Diode_SMD, F.Cu at (275.3, 70.0)
- added Ref**: Val**, kbd_Hole:m2_Spacer_Hole, F.Cu at (254.8, 114.1)
- added Ref**: Val**, kbd_Hole:m2_Spacer_Hole, F.Cu at (131.0, 96.5)
- added Ref**: Val**, kbd_Hole:m2_Spacer_Hole, F.Cu at (188.1, 96.5)
- added Ref**: Val**, kbd_Hole:m2_Spacer_Hole, F.Cu at (64.3, 114.1)
- added Ref**: Val**, kbd_Hole:m2_Spacer_Hole, F.Cu at (254.6, 60.0)
- added Ref**: Val**, kbd_Hole:m2_Spacer_Hole, F.Cu at (276.0, 81.2)
- added Ref**: Val**, kbd_Hole:m2_Spacer_Hole, F.Cu at (43.1, 81.2)
- added Ref**: Val**, kbd_Hole:m2_Spacer_Hole, F.Cu at (140.5, 60.0)
- added Ref**: Val**, kbd_Hole:m2_Spacer_Hole, F.Cu at (178.6, 60.0)
- added Ref**: Val**, kbd_Hole:m2_Spacer_Hole, F.Cu at (83.3, 60.0)
- added SW44: SW_Push, kbd_SW:CherryMX_Hotswap_1.5u, F.Cu at (264.3, 50.0)
- added SW45: SW_Push, kbd_SW:CherryMX_Hotswap_1.25u, F.Cu at (266.7, 69.1)
- D1, D10, D11, D12, D13, D14, D15, D16, D17, D18, D19, D2, D20, D21, D22, D23, D24, D25, D26, D27, D28, D29, D3, D30, D31, D32, D33, D34, D35, D36, D37, D38, D39, D4, D5, D6, D7, D8, D9: footprint kbd_Parts:Diode_TH_SMD -> kbd_Parts:Diode_SMD
- D40: renamed from D41; footprint kbd_Parts:Diode_TH_SMD -> kbd_Parts:Diode_SMD
- D42: renamed from D43; footprint kbd_Parts:Diode_TH_SMD -> kbd_Parts:Diode_SMD
- SW13, SW29, SW33, SW37, SW5, SW9: footprint kbd_SW:CherryMX_Hotswap_1u -> kbd_SW:CherryMX_Hotswap_1.25u
- SW4: footprint kbd_SW:CherryMX_Hotswap_1.5u -> kbd_SW:CherryMX_Hotswap_1.75u
- U1: moved to F.Cu
- moved SW42 23.8 mm to (245.3, 69.1)
- moved D36 22.3 mm to (275.3, 108.3), turned to 90 degrees
- moved SW43 21.3 mm to (262.0, 88.1)
- moved D42 17.3 mm to (271.0, 86.9)
- moved SW37 16.7 mm to (266.7, 107.2)
- moved SW1 13.7 mm to (45.2, 60.5), turned to 0 degrees
- moved D32 12.7 mm to (251.5, 108.3)
- moved SW33 11.9 mm to (242.9, 107.2)
- moved D28 8.19 mm to (227.7, 108.1)
- moved D4 7.61 mm to (61.0, 108.1), turned to 90 degrees
- moved SW5 7.14 mm to (52.4, 107.2)
- moved SW29 7.14 mm to (219.1, 107.2)
- moved D24 6.40 mm to (196.7, 108.1)
- moved D16 6.26 mm to (139.6, 108.1)
- moved D39 6.08 mm to (244.3, 89.1)
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- renumbered SW42 to SW41, SW43 to SW42, SW44 to SW43
Connections:
- U1 pad 10: Col0 -> Col1
- U1 pad 11: Col1 -> Col2
- U1 pad 12: Col2 -> Col3
- U1 pad 13: Col10 -> Col11
- U1 pad 14: Col9 -> Col10
- U1 pad 15: Col8 -> Col9
- U1 pad 16: Col7 -> Col8
- U1 pad 17: Col6 -> Col7
- U1 pad 18: Col5 -> Col6
- U1 pad 19: Col4 -> Col5
- U1 pad 20: Col3 -> Col4
- U1 pad 5: unconnected-(U1-D1/PIN5/SDA-Pad5) -> Row0
- U1 pad 6: Row0 -> Row1
- U1 pad 7: Row1 -> Row2
- U1 pad 8: Row2 -> Row3
- U1 pad 9: Row3 -> Col0
Routing:
- net Col11: track 0.00 -> 210.3 mm
- net Row2: track 277.0 -> 243.9 mm, vias 0 -> 17
- net Row3: track 299.5 -> 271.6 mm, vias 0 -> 1
- net Col9: track 220.0 -> 195.3 mm, vias 5 -> 1
- net Col3: track 119.6 -> 97.1 mm, vias 10 -> 0
- net Col8: track 220.9 -> 237.1 mm, vias 7 -> 0
- net Col0: track 97.0 -> 83.9 mm
- net Col7: track 205.1 -> 218.0 mm, vias 9 -> 1
- net Row1: track 266.6 -> 254.0 mm, vias 0 -> 13
- net Net-(D3-A): track 14.3 -> 5.50 mm
- net Net-(D4-A): track 13.9 -> 5.49 mm
- net Net-(D2-A): track 13.9 -> 5.50 mm
- net Net-(D40-A) (its old number): track 8.28 -> 0.00 mm
- net GND: track 45.0 -> 37.4 mm
- net Net-(D1-A): track 13.2 -> 5.83 mm
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Other:
- board size 229.6 x 78.6 mm -> 239.1 x 78.6 mm
