File: cr432/assemble/assemble.kicad_sch (KiCad schematic)
At the start: 88 parts, among them SW1 SW_Push, SW10 SW_Push, SW11 SW_Push, SW12 SW_Push, SW13 SW_Push, SW14 SW_Push, SW15 SW_Push, SW16 SW_Push, SW17 SW_Push, SW18 SW_Push, SW19 SW_Push, SW2 SW_Push, SW20 SW_Push, SW21 SW_Push, SW22 SW_Push, SW23 SW_Push, SW24 SW_Push, SW25 SW_Push, SW26 SW_Push, SW27 SW_Push, SW28 SW_Push, SW29 SW_Push, SW3 SW_Push, SW30 SW_Push, SW31 SW_Push, SW32 SW_Push, SW33 SW_Push, SW34 SW_Push, SW35 SW_Push, SW36 SW_Push, SW37 SW_Push, SW38 SW_Push, SW39 SW_Push, SW4 SW_Push, SW40 SW_Push, SW41 SW_Push, SW42 SW_Push, SW43 SW_Push, SW44 SW_Push, SW5 SW_Push, SW6 SW_Push, SW7 SW_Push, SW8 SW_Push, SW9 SW_Push, U1 Micon_BLEMicroPro

Commit message: rev1
Parts:
- removed D40: D, kbd_Parts:Diode_TH_SMD, symbol Device:D
- removed SW41: SW_Push, kbd_SW:CherryMX_Hotswap_1.5u, symbol Switch:SW_Push
- added D43, D44: D, kbd_Parts:Diode_SMD, symbol Device:D
- added SW44: SW_Push, kbd_SW:CherryMX_Hotswap_1.5u, symbol Switch:SW_Push
- added SW45: SW_Push, kbd_SW:CherryMX_Hotswap_1.25u, symbol Switch:SW_Push
- D1, D10, D11, D12, D13, D14, D15, D16, D17, D18, D19, D2, D20, D21, D22, D23, D24, D25, D26, D27, D28, D29, D3, D30, D31, D32, D33, D34, D35, D36, D37, D38, D39, D4, D5, D6, D7, D8, D9: footprint kbd_Parts:Diode_TH_SMD -> kbd_Parts:Diode_SMD
- D40: renamed from D41; footprint kbd_Parts:Diode_TH_SMD -> kbd_Parts:Diode_SMD
- D41: renamed from D42; footprint kbd_Parts:Diode_TH_SMD -> kbd_Parts:Diode_SMD
- D42: renamed from D43; footprint kbd_Parts:Diode_TH_SMD -> kbd_Parts:Diode_SMD
- SW13, SW29, SW33, SW37, SW5, SW9: footprint kbd_SW:CherryMX_Hotswap_1u -> kbd_SW:CherryMX_Hotswap_1.25u
- SW4: footprint kbd_SW:CherryMX_Hotswap_1.5u -> kbd_SW:CherryMX_Hotswap_1.75u
- renumbered SW42 to SW41, SW43 to SW42, SW44 to SW43
Connections:
- net Col0: now also U1.9 (D7/PIN9); no longer U1.10 (E6/PIN10)
- net Col1: now also U1.10 (E6/PIN10); no longer U1.11 (B4/PIN11)
- net Col10: now also U1.14 (B2/PIN14); no longer U1.13 (B6/PIN13)
- net Col2: now also U1.11 (B4/PIN11); no longer U1.12 (B5/PIN12)
- net Col3: now also U1.12 (B5/PIN12); no longer U1.20 (F4/PIN20)
- net Col4: now also U1.20 (F4/PIN20); no longer U1.19 (F5/PIN19)
- net Col5: now also U1.19 (F5/PIN19); no longer U1.18 (F6/PIN18)
- net Col6: now also U1.18 (F6/PIN18); no longer U1.17 (F7/PIN17)
- net Col7: now also U1.17 (F7/PIN17); no longer U1.16 (B1/PIN16)
- net Col8: now also U1.16 (B1/PIN16); no longer U1.15 (B3/PIN15)
- net Col9: now also U1.15 (B3/PIN15); no longer U1.14 (B2/PIN14)
- net Row0: now also U1.5 (D1/PIN5/SDA), D43.1 (K); no longer U1.6 (D0/PIN6/SCL)
- net Row1: now also U1.6 (D0/PIN6/SCL), D44.1 (K); no longer U1.7 (D4/PIN7)
- net Row2: now also U1.7 (D4/PIN7); no longer U1.8 (C6/PIN8)
- net Row3: now also U1.8 (C6/PIN8); no longer U1.9 (D7/PIN9)
- new net: D43.2 (A), SW44.2
- new net: D44.2 (A), SW45.2
- new net Col11: SW44.1, SW45.1, U1.13 (B6/PIN13)
- no-connect marks 5 -> 4
Other:
- moved on the sheet: D1, D10, D13, D14, D15, D16, D17, D18, D19, D2, D20, D21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
