File: cr432/bottom/bottom.kicad_pcb (KiCad board)
At the start: 2 copper layers, 229.6 x 78.6 mm, 0 parts

Commit message: rev1
Parts:
- added Ref**: Val**, kbd_Hole:m2_Screw_Hole, F.Cu at (172.1, 62.2)
- added Ref**: Val**, kbd_Hole:m2_Screw_Hole, F.Cu at (57.7, 116.3)
- added Ref**: Val**, kbd_Hole:m2_Screw_Hole, F.Cu at (133.9, 62.2)
- added Ref**: Val**, kbd_Hole:m2_Screw_Hole, F.Cu at (248.0, 62.2)
- added Ref**: Val**, kbd_Hole:m2_Screw_Hole, F.Cu at (36.6, 83.4)
- added Ref**: Val**, kbd_Hole:m2_Screw_Hole, F.Cu at (269.4, 83.4)
- added Ref**: Val**, kbd_Hole:m2_Screw_Hole, F.Cu at (181.6, 98.7)
- added Ref**: Val**, kbd_Hole:m2_Screw_Hole, F.Cu at (124.4, 98.7)
- added Ref**: Val**, kbd_Hole:m2_Screw_Hole, F.Cu at (76.8, 62.2)
- added Ref**: Val**, kbd_Hole:m2_Screw_Hole, F.Cu at (248.3, 116.3)
Other:
- board size 229.6 x 78.6 mm -> 239.1 x 78.6 mm
