File: cr432/top/top.kicad_pcb (KiCad board)
At the start: 2 copper layers, 229.6 x 78.6 mm, 57 parts, among them SW10 SW_Push, SW11 SW_Push, SW12 SW_Push, SW13 SW_Push, SW14 SW_Push, SW15 SW_Push, SW16 SW_Push, SW17 SW_Push, SW18 SW_Push, SW19 SW_Push, SW2 SW_Push, SW20 SW_Push, SW21 SW_Push, SW22 SW_Push, SW23 SW_Push, SW24 SW_Push, SW25 SW_Push, SW26 SW_Push, SW27 SW_Push, SW28 SW_Push, SW29 SW_Push, SW3 SW_Push, SW30 SW_Push, SW31 SW_Push, SW32 SW_Push, SW33 SW_Push, SW34 SW_Push, SW35 SW_Push, SW36 SW_Push, SW37 SW_Push, SW38 SW_Push, SW39 SW_Push, SW4 SW_Push, SW40 SW_Push, SW41 SW_Push, SW42 SW_Push, SW43 SW_Push, SW44 SW_Push, SW5 SW_Push, SW6 SW_Push, SW7 SW_Push, SW8 SW_Push, SW9 SW_Push

Commit message: rev1
Parts:
- removed the Ref** at (126.2, 79.3)
- removed the Ref** at (80.2, 42.1)
- removed the Ref** at (193.8, 42.1)
- removed the Ref** at (257.2, 115.0)
- removed the Ref** at (183.4, 79.3)
- removed the Ref** at (202.4, 115.0)
- removed the Ref** at (117.6, 42.1)
- removed the Ref** at (83.3, 77.9)
- removed the Ref** at (266.7, 95.2)
- removed the Ref** at (52.4, 115.0)
- removed the Ref** at (235.7, 77.9)
- removed the Ref** at (251.7, 42.1)
- removed the Ref** at (107.2, 115.0)
- removed the Ref** at (42.9, 95.2)
- added Ref**: Val**, kbd_Hole:m2_Screw_Hole, F.Cu at (245.3, 61.6)
- added Ref**: Val**, kbd_Hole:m2_Screw_Hole, F.Cu at (131.2, 61.6)
- added Ref**: Val**, kbd_Hole:m2_Screw_Hole, F.Cu at (266.7, 82.8)
- added Ref**: Val**, kbd_Hole:m2_Screw_Hole, F.Cu at (178.8, 98.1)
- added Ref**: Val**, kbd_Hole:m2_Screw_Hole, F.Cu at (245.5, 115.7)
- added Ref**: Val**, kbd_Hole:m2_Screw_Hole, F.Cu at (33.8, 82.8)
- added Ref**: Val**, kbd_Hole:m2_Screw_Hole, F.Cu at (55.0, 115.7)
- added Ref**: Val**, kbd_Hole:m2_Screw_Hole, F.Cu at (74.0, 61.6)
- added Ref**: Val**, kbd_Hole:m2_Screw_Hole, F.Cu at (169.3, 61.6)
- added Ref**: Val**, kbd_Hole:m2_Screw_Hole, F.Cu at (121.7, 98.1)
- added SW45: SW_Push, kbd_SW_Hole:SW_Hole_1.25u, F.Cu at (257.4, 70.7)
- SW13, SW29, SW33, SW37, SW5, SW9: footprint kbd_SW_Hole:SW_Hole_1u -> kbd_SW_Hole:SW_Hole_1.25u
- SW4: footprint kbd_SW_Hole:SW_Hole_1.5u -> kbd_SW_Hole:SW_Hole_1.75u
- SW41: footprint kbd_SW_Hole:SW_Hole_1.5u -> kbd_SW_Hole:SW_Hole_1u
- SW43: footprint kbd_SW_Hole:SW_Hole_1u -> kbd_SW_Hole:SW_Hole_1.75u
- SW44: footprint kbd_SW_Hole:SW_Hole_1.75u -> kbd_SW_Hole:SW_Hole_1.5u
- moved SW41 43.5 mm to (231.2, 51.6)
- moved SW43 40.3 mm to (252.7, 89.7)
- moved SW42 21.2 mm to (236.0, 70.7)
- moved SW44 17.6 mm to (255.0, 51.6)
- moved SW5 16.5 mm to (43.1, 108.8)
- moved SW9 11.8 mm to (66.9, 108.8)
- moved SW2 9.45 mm to (40.7, 51.6)
- moved SW10 9.45 mm to (78.8, 51.6)
- moved SW26 9.45 mm to (155.0, 51.6)
- moved SW6 9.45 mm to (59.8, 51.6)
- moved SW11 9.45 mm to (83.6, 70.7)
- moved SW14 9.45 mm to (97.8, 51.6)
- moved SW15 9.45 mm to (102.6, 70.7)
- moved SW19 9.45 mm to (121.7, 70.7)
- moved SW22 9.45 mm to (135.9, 51.6)
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Other:
- board size 229.6 x 78.6 mm -> 239.1 x 78.6 mm
